File: keyboard_proj/battery.kicad_sch (KiCad schematic)
At the start: 17 parts, among them IC1 DW01A-G, IC2 TP4056-42-ESOP8, IC3 LD1117DT12CTR, Q1 FS8205A, Q2 2N7002, U7 SK12D07VG5, U9 1.0K-ES-4PWB

Commit message: PCB bien avancé, presque fini mais je dois selectionner des pieces de jlcpcb pour baisser les couts
Parts:
- C6: value 100 uF -> 100nF; LCSC (none) -> C880603
- C7, C_out_LDO1: LCSC (none) -> C723895
- C_in_LDO1: LCSC (none) -> C880603
- IC1: LCSC (none) -> C436931
- IC2: LCSC (none) -> C16581
- IC3: LCSC (none) -> C36395
- Q1: LCSC (none) -> C2830320
- Q2: LCSC (none) -> C916396
- R28: value 500 -> 1kΩ; LCSC (none) -> C2909306
- R29: value 300 -> 300Ω; LCSC (none) -> C1882580
- R3: value 1k -> 1kΩ; LCSC (none) -> C2909306
- R4: value 1.2k -> 1kΩ; LCSC (none) -> C2909306
- R5: value 100 -> 100Ω; LCSC (none) -> C304972
- U7: LCSC (none) -> C431548
- U9: LCSC (none) -> C2915277
